File: Electronics/Electronics.kicad_sch (KiCad schematic)
At the start: 88 parts

Commit message: PCB finished with Gerbers
Parts:
- C1, C2, C3, C4, C5, C6, C7: renamed from C?; footprint (none) -> Capacitor_SMD:C_0805_2012Metric
- D1, D10, D11, D12, D13, D14, D15, D16, D17, D18, D19, D2, D20, D21, D22, D23, D24, D25, D26, D27, D28, D29, D3, D30, D31, D32, D33, D34, D35, D36, D4, D5, D6, D7, D8, D9: renamed from D?; footprint (none) -> Diode_SMD:D_SOD-123
- F1: renamed from F?; footprint (none) -> Fuse:Fuse_1206_3216Metric
- MX1, MX10, MX11, MX12, MX13, MX14, MX15, MX16, MX17, MX18, MX19, MX2, MX20, MX21, MX22, MX23, MX24, MX25, MX26, MX27, MX28, MX29, MX3, MX30, MX31, MX32, MX33, MX34, MX35, MX36, MX4, MX5, MX6, MX7, MX8, MX9: renamed from MX?; footprint (none) -> MX_Alps_Hybrid:MX-1U-NoLED
- R1, R2, R3, R4: renamed from R?; footprint (none) -> Resistor_SMD:R_0805_2012Metric
- SW1: renamed from SW?; footprint (none) -> random-keyboard-parts:SKQG-1155865
- USB1: renamed from USB?; footprint (none) -> random-keyboard-parts:Molex-0548190589
- Y1: renamed from Y?; footprint (none) -> Crystal:Crystal_SMD_3225-4Pin_3.2x2.5mm
- gave numbers to parts that had none: 1
Connections:
- net COL0: now also U1.37 (PF6); no longer U1.8 (PB0)
- net COL1: now also U1.36 (PF7); no longer U1.9 (PB1)
- net COL10: now also U1.20 (PD2); no longer U1.18 (PD0)
- net COL2: now also U1.32 (PC7); no longer U1.10 (PB2)
- net COL3: now also U1.31 (PC6); no longer U1.11 (PB3)
- net COL4: now also U1.30 (PB6); no longer U1.28 (PB4)
- net COL5: now also U1.19 (PD1); no longer U1.29 (PB5)
- net COL6: now also U1.26 (PD6); no longer U1.30 (PB6)
- net COL7: now also U1.25 (PD4); no longer U1.12 (PB7)
- net COL8: now also U1.22 (PD5); no longer U1.31 (PC6)
- net COL9: now also U1.21 (PD3); no longer U1.32 (PC7)
- net ROW0: now also U1.29 (PB5); no longer U1.19 (PD1)
- net ROW1: now also U1.28 (PB4); no longer U1.20 (PD2)
- net ROW2: now also U1.27 (PD7); no longer U1.21 (PD3)
- net ROW3: now also U1.18 (PD0); no longer U1.25 (PD4)
